Commit message: new_engineer

File: moveit_config/config/gazebo_engineer_framed.urdf (robot description, URDF)
Before this commit: robot engineer_framed, 13 links, 12 joints
Links:
- removed link link1_br
- removed link link2_bl
- removed link link3_fr
- removed link link4_fl
- added link link1_fl, mass 0.70318; collision mesh filename=package://sp_description/meshes/engineer_framed/engineer_ch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; visual mesh filename=package://sp_description/meshes/engineer_framed/engineer_ch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
- added link link2_fr, mass 0.69776; collision mesh filename=package://sp_description/meshes/engineer_framed/engineer_ch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; visual mesh filename=package://sp_description/meshes/engineer_framed/engineer_ch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
- added link link3_bl, mass 0.68237; collision mesh filename=package://sp_description/meshes/engineer_framed/engineer_ch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; visual mesh filename=package://sp_description/meshes/engineer_framed/engineer_ch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
- added link link4_br, mass 0.70951; collision mesh filename=package://sp_description/meshes/engineer_framed/engineer_ch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; visual mesh filename=package://sp_description/meshes/engineer_framed/engineer_ch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
- link arm_base_link: mass 1.851 -> 3.4509
- link base_link: mass 6.2008 -> 6.3166
- link link1: mass 3.3269 -> 3.3312
- link link3: mass 0.53637 -> 0.53167
- link link4: mass 1.4781 -> 2.56
- link link6: mass 0.66912 -> 0.63735
Joints:
- removed joint joint1_br
- removed joint joint2_bl
- removed joint joint3_fr
- removed joint joint4_fl
- added joint joint1_fl: type continuous, parent base_link, child link1_fl, origin xyz=-0.24531 -0.3683 -0.05551 rpy=1.5708 -0.088599 -1.5708, axis 0 0 -1
- added joint joint2_fr: type continuous, parent base_link, child link2_fr, origin xyz=0.11159 -0.3683 -0.05551 rpy=-1.5708 -0.81082 -1.5708, axis 0 0 1
- added joint joint3_bl: type continuous, parent base_link, child link3_bl, origin xyz=-0.20121 -0.7517 -0.05551 rpy=1.5708 0.8753 -1.5708, axis 0 0 1, limit lower=0 upper=0 effort=0 velocity=0
- added joint joint4_br: type continuous, parent base_link, child link4_br, origin xyz=0.15569 -0.75167 -0.055404 rpy=1.5708 -0.089686 1.5708, axis 0 0 1
- joint joint1: limit lower=-0.3012 upper=0 effort=0 velocity=0 -> lower=-0.3012 upper=0 effort=20 velocity=6
- joint joint2: limit lower=0 upper=0.4394 effort=0 velocity=0 -> lower=0 upper=0.86634 effort=20 velocity=6; origin xyz=-0.27 0 0.4126 rpy=0 0 0 -> xyz=-0.273 0 0.3831 rpy=0 0 0
- joint joint3: limit lower=0 upper=0.4754 effort=0 velocity=0 -> lower=0 upper=0.4754 effort=20 velocity=6; origin xyz=0.42494 0 0.042 rpy=0 0 0 -> xyz=0.42794 0 0.072 rpy=0 0 0
- joint joint4: limit lower=-0.017022 upper=0.013858 effort=0 velocity=0 -> lower=-0.4 upper=0.4 effort=20 velocity=6
- joint joint5: axis 0 0 -1 -> 0 0 1; limit lower=0 upper=3.14 effort=0 velocity=0 -> lower=0 upper=3.14 effort=20 velocity=6; origin xyz=0 -0.007 0.128 rpy=-1.5708 0 0 -> xyz=0 -0.019 0.128 rpy=1.5708 0 0
- joint joint6: limit lower=-1.57 upper=+1.57 effort=0 velocity=0 -> lower=-1.57 upper=1.57 effort=20 velocity=6; origin xyz=0.071794 0 0.028 rpy=-1.5708 0 -1.5708 -> xyz=0.071794 0 -0.028 rpy=0 1.5708 0
- joint joint7: limit lower=-1.57 upper=+1.57 effort=0 velocity=0 -> lower=-1.57 upper=1.57 effort=20 velocity=6; origin xyz=0.18801 0.00015076 -0.071797 rpy=0 -1.5708 0 -> xyz=0 0.17579 -0.071794 rpy=1.5708 0 3.1416
- joint joint_arm2body: origin xyz=0.011757 0.00020017 -0.0013475 rpy=0 0 1.57 -> xyz=-0.044504 -0.55819 -0.012391 rpy=0 0 0

File: sp_description/urdf/engineer_framed/engineer_framed.xacro (robot description, xacro)
@@ -2,19 +2,22 @@
 <robot xmlns:xacro="http://www.ros.org/wiki/xacro" name="engineer_framed">
 	<xacro:include filename="$(find sp_description)/urdf/engineer_framed/engineer_manipulator_framed/engineer_manipulator_framed.xacro"/>
-	<xacro:include filename="$(find sp_description)/urdf/engineer_framed/engineer_chassis/engineer_chassis.xacro"/>
-	<xacro:include filename="$(find sp_description)/urdf/engineer_framed/manipulator_transmission.xacro"/>
+	<xacro:include filename="$(find sp_description)/urdf/engineer_framed/engineer_chassis_framed/engineer_chassis_framed.xacro"/>
+	<xacro:include filename="$(find sp_description)/urdf/engineer_manipulator/manipulator_transmission.xacro"/>
     <xacro:engineer_manipulator_framed/>
-    <xacro:engineer_chassis roller_type="simple"/>
+    <xacro:engineer_chassis_framed roller_type="simple"/>
+	<!-- <link name="world" />
+	<xacro:engineer_chassis_framed xyz="0 0 0" rpy="0 0 0" connected_to="world"/> -->
+	<xacro:arg name="use_simulation" default="true"/>
     	<joint name="joint_arm2body" type="fixed">
 		<axis xyz="0 0 1"/>
-		<origin xyz="0.011757 0.00020017 -0.0013475" rpy="0 0 1.57"/>
+		<origin xyz="-0.044504 -0.55819 -0.012391" rpy="0 0 0"/>
 		<parent link="base_link"/>
 		<child link="arm_base_link"/>
 	</joint>
-	<!--在机器人模型的urdf/xacro文件中添加gazebo_ros_control插件-->
+		<!--在机器人模型的urdf/xacro文件中添加gazebo_ros_control插件-->
 	<gazebo>
 		<plugin name="gazebo_ros_control" filename="libgazebo_ros_control.so">
-			<robotNamespace>/engineer_framed</robotNamespace>
+			<robotNamespace>/</robotNamespace>
 		</plugin>
 		</gazebo>
-</robot>
+    </robot>

File: sp_description/urdf/engineer_framed/engineer_manipulator_framed/engineer_manipulator_framed.xacro (robot description, xacro)
@@ -11,15 +11,15 @@
     <inertial>
       <origin
-        xyz="-0.037522 -0.068476 0.28458"
-        rpy="0 0 0" />
-      <mass
-        value="1.851" />
-      <inertia
-        ixx="0.013502"
-        ixy="1.5471E-07"
-        ixz="-1.0797E-06"
-        iyy="0.013899"
-        iyz="2.8303E-07"
-        izz="0.00075044" />
+        xyz="-0.02624 -0.018282 0.25067"
+        rpy="0 0 0" />
+      <mass
+        value="3.4509" />
+      <inertia
+        ixx="0.030137"
+        ixy="-1.2844E-07"
+        ixz="-3.1208E-06"
+        iyy="0.030724"
+        iyz="3.4634E-08"
+        izz="0.0009827" />
     </inertial>
     <visual>
@@ -51,15 +51,15 @@
     <inertial>
       <origin
-        xyz="-0.046385 -0.011064 0.39469"
-        rpy="0 0 0" />
-      <mass
-        value="3.3269" />
-      <inertia
-        ixx="0.0042506"
+        xyz="-0.046418 -0.011017 0.39513"
+        rpy="0 0 0" />
+      <mass
+        value="3.3312" />
+      <inertia
+        ixx="0.0042512"
         ixy="-2.4588E-07"
-        ixz="4.5157E-06"
-        iyy="0.047094"
+        ixz="4.5056E-06"
+        iyy="0.047104"
         iyz="-5.1474E-08"
-        izz="0.050675" />
+        izz="0.050684" />
     </inertial>
     <visual>
@@ -100,8 +100,8 @@
       xyz="0 0 1" />
     <limit
-      lower="-0.3012"
+      lower="-0.2012"
       upper="0"
-      effort="0"
-      velocity="0" />
+      effort="20"
+      velocity="6" />
   </joint>
   <link
@@ -109,5 +109,5 @@
     <inertial>
       <origin
-        xyz="0.73463 -0.012605 0.039937"
+        xyz="0.73763 -0.012605 0.269937"
         rpy="0 0 0" />
       <mass
@@ -149,5 +149,5 @@
     type="prismatic">
     <origin
-      xyz="-0.27 0 0.4126"
+      xyz="-0.273 0 0.3831"
       rpy="0 0 0" />
     <parent
@@ -159,7 +159,7 @@
     <limit
       lower="0"
-      upper="0.4394"
-      effort="0"
-      velocity="0" />
+      upper="0.86634"
+      effort="20"
+      velocity="6" />
   </joint>
   <link
@@ -167,15 +167,15 @@
     <inertial>
       <origin
-        xyz="0.51092 0.0050158 0.038576"
-        rpy="0 0 0" />
-      <mass
-        value="0.53637" />
-      <inertia
-        ixx="0.006721"
-        ixy="-1.2751E-06"
-        ixz="5.8146E-09"
-        iyy="0.00010173"
-        iyz="3.4689E-08"
-        izz="0.0067953" />
+        xyz="0.51093 0.000566 0.038621"
+        rpy="0 0 0" />
+      <mass
+        value="0.53167" />
+      <inertia
+        ixx="0.0064934"
+        ixy="-2.3958E-07"
+        ixz="8.5458E-09"
+        iyy="9.996E-05"
+        iyz="2.0423E-08"
+        izz="0.0065666" />
     </inertial>
     <visual>
@@ -207,5 +207,5 @@
     type="prismatic">
     <origin
-      xyz="0.42494 0 0.042"
+      xyz="0.42794 0 0.072"
       rpy="0 0 0" />
     <parent
@@ -218,6 +218,6 @@
       lower="0"
       upper="0.4754"
-      effort="0"
-      velocity="0" />
+      effort="20"
+      velocity="6" />
   </joint>
   <link
@@ -225,15 +225,15 @@
     <inertial>
       <origin
-        xyz="-0.004492 0.0012594 0.076929"
-        rpy="0 0 0" />
-      <mass
-        value="1.4781" />
-      <inertia
-        ixx="0.00699"
-        ixy="-4.5494E-07"
-        ixz="-1.6934E-07"
-        iyy="0.00040962"
-        iyz="-2.7173E-07"
-        izz="0.006972" />
+        xyz="0.0022176 0.055912 0.11366"
+        rpy="0 0 0" />
+      <mass
+        value="2.56" />
+      <inertia
+        ixx="0.0074237"
+        ixy="-1.2559E-06"
+        ixz="-6.9104E-06"
+        iyy="0.00083452"
+        iyz="-5.1569E-07"
+        izz="0.0075779" />
     </inertial>
     <visual>
@@ -274,8 +274,8 @@
       xyz="0 1 0" />
     <limit
-      lower="-0.17022"
-      upper="0.13858"
-      effort="0"
-      velocity="0" />
+      lower="-0.185"
+      upper="0.185"
+      effort="20"
+      velocity="6" />
   </joint>
   <link
@@ -283,5 +283,5 @@
     <inertial>
       <origin
-        xyz="0.037482 -0.0011554 0.028017"
+        xyz="0.037482 0.0011554 -0.028017"
         rpy="0 0 0" />
       <mass
@@ -289,6 +289,6 @@
       <inertia
         ixx="0.00016271"
-        ixy="1.8762E-07"
-        ixz="1.4951E-07"
+        ixy="-1.8762E-07"
+        ixz="-1.4951E-07"
         iyy="9.8184E-05"
         iyz="4.2357E-09"
@@ -323,6 +323,6 @@
     type="revolute">
     <origin
-      xyz="0 -0.007 0.128"
-      rpy="-1.5708 0 0" />
+      xyz="0 -0.019 0.128"
+      rpy="1.5708 0 0" />
     <parent
       link="link4" />
@@ -330,10 +330,10 @@
       link="link5" />
     <axis
-      xyz="0 0 -1" />
+      xyz="0 0 1" />
     <limit
       lower="0"
       upper="3.14"
-      effort="0"
-      velocity="0" />
+      effort="20"
+      velocity="6" />
   </joint>
   <link
@@ -341,15 +341,15 @@
     <inertial>
       <origin
-        xyz="0.14216 -0.00011579 -0.0086719"
-        rpy="0 0 0" />
-      <mass
-        value="0.66912" />
-      <inertia
-        ixx="0.00027285"
-        ixy="1.2504E-08"
-        ixz="2.9576E-06"
-        iyy="0.00027332"
-        iyz="-2.2374E-07"
-        izz="0.00025157" />
+        xyz="0.0001049 0.14059 -0.0055479"
+        rpy="0 0 0" />
+      <mass
+        value="0.63735" />
+      <inertia
+        ixx="0.00027146"
+        ixy="1.1047E-08"
+        ixz="2.2272E-07"
+        iyy="0.00027079"
+        iyz="2.9582E-06"
+        izz="0.0002496" />
     </inertial>
     <visual>
@@ -381,6 +381,6 @@
     type="revolute">
     <origin
-      xyz="0.071794 0 0.028"
-      rpy="-1.5708 0 -1.5708" />
+      xyz="0.071794 0 -0.028"
+      rpy="0 1.5708 0" />
     <parent
       link="link5" />
@@ -391,7 +391,7 @@
     <limit
       lower="-1.57"
-      upper="+1.57"
-      effort="0"
-      velocity="0" />
+      upper="1.57"
+      effort="20"
+      velocity="6" />
   </joint>
   <link
@@ -399,14 +399,14 @@
     <inertial>
       <origin
-        xyz="-0.057503 0.0014691 0.022736"
+        xyz="-0.0013183 -0.057506 0.034955"
         rpy="0 0 0" />
       <mass
         value="0.19723" />
       <inertia
-        ixx="6.2669E-05"
-        ixy="1.059E-06"
-        ixz="3.9133E-08"
-        iyy="0.00010859"
-        iyz="-2.4478E-08"
+        ixx="0.00010859"
+        ixy="-1.059E-06"
+        ixz="2.4478E-08"
+        iyy="6.2669E-05"
+        iyz="3.9133E-08"
         izz="0.00015495" />
     </inertial>
@@ -439,6 +439,6 @@
     type="revolute">
     <origin
-      xyz="0.18801 0.00015076 -0.071797"
-      rpy="0 -1.5708 0" />
+      xyz="0 0.17579 -0.071794"
+      rpy="1.5708 0 3.1416" />
     <parent
       link="link6" />
@@ -449,8 +449,8 @@
     <limit
       lower="-1.57"
-      upper="+1.57"
-      effort="0"
-      velocity="0" />
-  </joint>
-  </xacro:macro>
+      upper="1.57"
+      effort="20"
+      velocity="6" />
+  </joint>
+   </xacro:macro>
 </robot>

File: sp_description/urdf/engineer_manipulator/manipulator_transmission.xacro (robot description, xacro)
@@ -20,5 +20,5 @@
     <xacro:manipulator_transmission joint_name="joint6" mechanical_reduction="1"/>
     <xacro:manipulator_transmission joint_name="joint7" mechanical_reduction="599.99"/>
-    <gazebo>
+    <!-- <gazebo>
         <plugin name="gazebo_ros_vacuum_gripper" filename="libgazebo_ros_vacuum_gripper.so">
             <robotNamespace>/vacuum_gripper</robotNamespace>
@@ -40,3 +40,4 @@
         <material>Gazebo/Grey</material>
     </gazebo>
+	 -->
 </robot>
