Commit message: new_engineer

File: moveit_config/config/gazebo_engineer_framed.urdf (robot description, URDF)
Before this commit: robot engineer_framed, 13 links, 12 joints
Links:
- removed link base_link
- removed link link1_fl
- removed link link2_fr
- removed link link3_bl
- removed link link4_br
- added link world
Joints:
- removed joint joint1_fl
- removed joint joint2_fr
- removed joint joint3_bl
- removed joint joint4_br
- removed joint joint_arm2body
- added joint world_joint: type fixed, parent world, child arm_base_link, origin xyz=0.0 0.0 0.0 rpy=0.0 0.0 0.0
- joint joint1: limit lower=-0.3012 upper=0 effort=20 velocity=6 -> lower=-0.3012 upper=0 effort=0 velocity=0
- joint joint2: limit lower=0 upper=0.86634 effort=20 velocity=6 -> lower=0 upper=0.86634 effort=0 velocity=0
- joint joint3: limit lower=0 upper=0.4754 effort=20 velocity=6 -> lower=0 upper=0.4754 effort=0 velocity=0
- joint joint4: limit lower=-0.4 upper=0.4 effort=20 velocity=6 -> lower=-0.4 upper=0.4 effort=0 velocity=0
- joint joint5: limit lower=0 upper=3.14 effort=20 velocity=6 -> lower=0 upper=3.14 effort=0 velocity=0
- joint joint6: limit lower=-1.57 upper=1.57 effort=20 velocity=6 -> lower=-1.57 upper=1.57 effort=0 velocity=0
- joint joint7: limit lower=-1.57 upper=1.57 effort=20 velocity=6 -> lower=-1.57 upper=1.57 effort=0 velocity=0

File: sp_description/urdf/engineer_framed/engineer_chassis_framed/engineer_chassis_framed.xacro (robot description, xacro)
@@ -7,18 +7,18 @@
   xmlns:xacro="http://wiki.ros.org/xacro">
   <xacro:macro name="engineer_chassis_framed" params="roller_type">
-  <link
+ <link
     name="base_link">
     <inertial>
       <origin
-        xyz="-0.044504 -0.55819 -0.012391"
+        xyz="-0.0018086 0.00030067 0.12012"
         rpy="0 0 0" />
       <mass
         value="6.3166" />
       <inertia
-        ixx="0.040448"
-        ixy="5.3584E-06"
-        ixz="-4.9021E-09"
-        iyy="0.02453"
-        iyz="-1.0636E-06"
+        ixx="0.02453"
+        ixy="-5.3584E-06"
+        ixz="1.0636E-06"
+        iyy="0.040448"
+        iyz="-4.9021E-09"
         izz="0.060871" />
     </inertial>
@@ -48,5 +48,5 @@
   </link>
   <link
-    name="link1_fl">
+    name="link1_br">
     <inertial>
       <origin
@@ -69,140 +69,140 @@
       <geometry>
         <mesh
-          filename="package://sp_description/meshes/engineer_framed/engineer_chassis/link1_fl.STL" />
-      </geometry>
-      <material
-        name="">
-        <color
-          rgba="0.69804 0.69804 0.69804 1" />
-      </material>
-    </visual>
-    <collision>
-      <origin
-        xyz="0 0 0"
-        rpy="0 0 0" />
-      <geometry>
-        <mesh
-          filename="package://sp_description/meshes/engineer_framed/engineer_chassis/link1_fl.STL" />
-      </geometry>
-    </collision>
-  </link>
-  <joint
-    name="joint1_fl"
-    type="continuous">
-    <origin
-      xyz="-0.24531 -0.3683 -0.05551"
-      rpy="1.5708 -0.088599 -1.5708" />
-    <parent
-      link="base_link" />
-    <child
-      link="link1_fl" />
+          filename="package://sp_description/meshes/engineer_framed/engineer_chassis/link1_br.STL" />
+      </geometry>
+      <material
+        name="">
+        <color
+          rgba="0.69804 0.69804 0.69804 1" />
+      </material>
+    </visual>
+    <collision>
+      <origin
+        xyz="0 0 0"
+        rpy="0 0 0" />
+      <geometry>
+        <mesh
+          filename="package://sp_description/meshes/engineer_framed/engineer_chassis/link1_br.STL" />
+      </geometry>
+    </collision>
+  </link>
+  <joint
+    name="joint1_br"
+    type="continuous">
+    <origin
+      xyz="-0.1917 -0.2005 0.077"
+      rpy="1.5708 -0.088599 0" />
+    <parent
+      link="base_link" />
+    <child
+      link="link1_br" />
     <axis
       xyz="0 0 -1" />
   </joint>
   <link
-    name="link2_fr">
-    <inertial>
-      <origin
-        xyz="-0.00051287 0.00030252 0.067842"
+    name="link2_bl">
+    <inertial>
+      <origin
+        xyz="-0.00013404 0.023742 -0.00058016"
         rpy="0 0 0" />
       <mass
         value="0.69776" />
       <inertia
-        ixx="0.0011572"
-        ixy="1.4786E-09"
-        ixz="-6.9974E-12"
-        iyy="0.0011718"
-        iyz="1.7156E-09"
-        izz="0.0022157" />
-    </inertial>
-    <visual>
-      <origin
-        xyz="0 0 0"
-        rpy="0 0 0" />
-      <geometry>
-        <mesh
-          filename="package://sp_description/meshes/engineer_framed/engineer_chassis/link2_fr.STL" />
-      </geometry>
-      <material
-        name="">
-        <color
-          rgba="0.69804 0.69804 0.69804 1" />
-      </material>
-    </visual>
-    <collision>
-      <origin
-        xyz="0 0 0"
-        rpy="0 0 0" />
-      <geometry>
-        <mesh
-          filename="package://sp_description/meshes/engineer_framed/engineer_chassis/link2_fr.STL" />
-      </geometry>
-    </collision>
-  </link>
-  <joint
-    name="joint2_fr"
-    type="continuous">
-    <origin
-      xyz="0.11159 -0.3683 -0.05551"
-      rpy="-1.5708 -0.81082 -1.5708" />
-    <parent
-      link="base_link" />
-    <child
-      link="link2_fr" />
-    <axis
-      xyz="0 0 1" />
-  </joint>
-  <link
-    name="link3_bl">
-    <inertial>
-      <origin
-        xyz="0.00042861 -4.5394E-05 0.068188"
+        ixx="0.0011649"
+        ixy="1.2388E-09"
+        ixz="-7.2836E-06"
+        iyy="0.0022157"
+        iyz="-1.187E-09"
+        izz="0.0011641" />
+    </inertial>
+    <visual>
+      <origin
+        xyz="0 0 0"
+        rpy="0 0 0" />
+      <geometry>
+        <mesh
+          filename="package://sp_description/meshes/engineer_framed/engineer_chassis/link2_bl.STL" />
+      </geometry>
+      <material
+        name="">
+        <color
+          rgba="0.69804 0.69804 0.69804 1" />
+      </material>
+    </visual>
+    <collision>
+      <origin
+        xyz="0 0 0"
+        rpy="0 0 0" />
+      <geometry>
+        <mesh
+          filename="package://sp_description/meshes/engineer_framed/engineer_chassis/link2_bl.STL" />
+      </geometry>
+    </collision>
+  </link>
+  <joint
+    name="joint2_bl"
+    type="continuous">
+    <origin
+      xyz="-0.1917 0.2005 0.077"
+      rpy="0 0 0" />
+    <parent
+      link="base_link" />
+    <child
+      link="link2_bl" />
+    <axis
+      xyz="0 1 0" />
+  </joint>
+  <link
+    name="link3_fr">
+    <inertial>
+      <origin
+        xyz="0.00023979 -0.024088 -0.00035815"
         rpy="0 0 0" />
       <mass
         value="0.68237" />
       <inertia
-        ixx="0.0011484"
-        ixy="1.4786E-09"
-        ixz="-6.9966E-12"
-        iyy="0.001163"
-        iyz="1.7156E-09"
-        izz="0.0021982" />
-    </inertial>
-    <visual>
-      <origin
-        xyz="0 0 0"
-        rpy="0 0 0" />
-      <geometry>
-        <mesh
-          filename="package://sp_description/meshes/engineer_framed/engineer_chassis/link3_bl.STL" />
-      </geometry>
-      <material
-        name="">
-        <color
-          rgba="0.69804 0.69804 0.69804 1" />
-      </material>
-    </visual>
-    <collision>
-      <origin
-        xyz="0 0 0"
-        rpy="0 0 0" />
-      <geometry>
-        <mesh
-          filename="package://sp_description/meshes/engineer_framed/engineer_chassis/link3_bl.STL" />
-      </geometry>
-    </collision>
-  </link>
-  <joint
-    name="joint3_bl"
-    type="continuous">
-    <origin
-      xyz="-0.20121 -0.7517 -0.05551"
-      rpy="1.5708 0.8753 -1.5708" />
-    <parent
-      link="base_link" />
-    <child
-      link="link3_bl" />
-    <axis
-      xyz="0 0 1" />
+        ixx="0.001157"
+        ixy="-1.3127E-09"
+        ixz="7.1752E-06"
+        iyy="0.0021982"
+        iyz="-1.1047E-09"
+        izz="0.0011544" />
+    </inertial>
+    <visual>
+      <origin
+        xyz="0 0 0"
+        rpy="0 0 0" />
+      <geometry>
+        <mesh
+          filename="package://sp_description/meshes/engineer_framed/engineer_chassis/link3_fr.STL" />
+      </geometry>
+      <material
+        name="">
+        <color
+          rgba="0.69804 0.69804 0.69804 1" />
+      </material>
+    </visual>
+    <collision>
+      <origin
+        xyz="0 0 0"
+        rpy="0 0 0" />
+      <geometry>
+        <mesh
+          filename="package://sp_description/meshes/engineer_framed/engineer_chassis/link3_fr.STL" />
+      </geometry>
+    </collision>
+  </link>
+  <joint
+    name="joint3_fr"
+    type="continuous">
+    <origin
+      xyz="0.1917 -0.2005 0.077"
+      rpy="0 0 0" />
+    <parent
+      link="base_link" />
+    <child
+      link="link3_fr" />
+    <axis
+      xyz="0 -1 0" />
     <limit
       lower="0"
@@ -212,55 +212,55 @@
   </joint>
   <link
-    name="link4_br">
-    <inertial>
-      <origin
-        xyz="0.00020184 -4.3664E-06 0.023775"
+    name="link4_fl">
+    <inertial>
+      <origin
+        xyz="-0.00020142 0.023775 1.3729E-05"
         rpy="0 0 0" />
       <mass
         value="0.70951" />
       <inertia
-        ixx="0.0011574"
-        ixy="1.4786E-09"
-        ixz="-6.9966E-12"
-        iyy="0.001172"
-        iyz="1.7156E-09"
-        izz="0.0022157" />
-    </inertial>
-    <visual>
-      <origin
-        xyz="0 0 0"
-        rpy="0 0 0" />
-      <geometry>
-        <mesh
-          filename="package://sp_description/meshes/engineer_framed/engineer_chassis/link4_br.STL" />
-      </geometry>
-      <material
-        name="">
-        <color
-          rgba="0.69804 0.69804 0.69804 1" />
-      </material>
-    </visual>
-    <collision>
-      <origin
-        xyz="0 0 0"
-        rpy="0 0 0" />
-      <geometry>
-        <mesh
-          filename="package://sp_description/meshes/engineer_framed/engineer_chassis/link4_br.STL" />
-      </geometry>
-    </collision>
-  </link>
-  <joint
-    name="joint4_br"
-    type="continuous">
-    <origin
-      xyz="0.15569 -0.75167 -0.055404"
-      rpy="1.5708 -0.089686 1.5708" />
-    <parent
-      link="base_link" />
-    <child
-      link="link4_br" />
-    <axis
-      xyz="0 0 1" />
+        ixx="0.0011576"
+        ixy="1.6063E-10"
+        ixz="1.2997E-06"
+        iyy="0.0022157"
+        iyz="1.7081E-09"
+        izz="0.0011719" />
+    </inertial>
+    <visual>
+      <origin
+        xyz="0 0 0"
+        rpy="0 0 0" />
+      <geometry>
+        <mesh
+          filename="package://sp_description/meshes/engineer_framed/engineer_chassis/link4_fl.STL" />
+      </geometry>
+      <material
+        name="">
+        <color
+          rgba="0.69804 0.69804 0.69804 1" />
+      </material>
+    </visual>
+    <collision>
+      <origin
+        xyz="0 0 0"
+        rpy="0 0 0" />
+      <geometry>
+        <mesh
+          filename="package://sp_description/meshes/engineer_framed/engineer_chassis/link4_fl.STL" />
+      </geometry>
+    </collision>
+  </link>
+  <joint
+    name="joint4_fl"
+    type="continuous">
+    <origin
+      xyz="0.19167 0.2005 0.077106"
+      rpy="0 0 0" />
+    <parent
+      link="base_link" />
+    <child
+      link="link4_fl" />
+    <axis
+      xyz="0 1 0" />
   </joint>
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
File: sp_description/urdf/engineer_framed/engineer_framed.xacro (robot description, xacro)
@@ -2,22 +2,8 @@
 <robot xmlns:xacro="http://www.ros.org/wiki/xacro" name="engineer_framed">
 	<xacro:include filename="$(find sp_description)/urdf/engineer_framed/engineer_manipulator_framed/engineer_manipulator_framed.xacro"/>
-	<xacro:include filename="$(find sp_description)/urdf/engineer_framed/engineer_chassis_framed/engineer_chassis_framed.xacro"/>
+	<!-- <xacro:include filename="$(find sp_description)/urdf/engineer_framed/engineer_chassis_framed/engineer_chassis_framed.xacro"/> -->
 	<xacro:include filename="$(find sp_description)/urdf/engineer_manipulator/manipulator_transmission.xacro"/>
     <xacro:engineer_manipulator_framed/>
-    <xacro:engineer_chassis_framed roller_type="simple"/>
-	<!-- <link name="world" />
-	<xacro:engineer_chassis_framed xyz="0 0 0" rpy="0 0 0" connected_to="world"/> -->
+    <!-- <xacro:engineer_chassis_framed roller_type="simple"/> -->
 	<xacro:arg name="use_simulation" default="true"/>
-    	<joint name="joint_arm2body" type="fixed">
-		<axis xyz="0 0 1"/>
-		<origin xyz="-0.044504 -0.55819 -0.012391" rpy="0 0 0"/>
-		<parent link="base_link"/>
-		<child link="arm_base_link"/>
-	</joint>
-		<!--在机器人模型的urdf/xacro文件中添加gazebo_ros_control插件-->
-	<gazebo>
-		<plugin name="gazebo_ros_control" filename="libgazebo_ros_control.so">
-			<robotNamespace>/</robotNamespace>
-		</plugin>
-		</gazebo>
     </robot>

File: sp_description/urdf/engineer_framed/engineer_manipulator_framed/engineer_manipulator_framed.xacro (robot description, xacro)
@@ -100,7 +100,7 @@
       xyz="0 0 1" />
     <limit
-      lower="-0.2012"
+       lower="-0.3012"
       upper="0"
-      effort="20"
+      effort="2000"
       velocity="6" />
   </joint>
@@ -109,5 +109,5 @@
     <inertial>
       <origin
-        xyz="0.73763 -0.012605 0.269937"
+        xyz="0.73763 -0.012605 0.069937"
         rpy="0 0 0" />
       <mass
@@ -160,5 +160,5 @@
       lower="0"
       upper="0.86634"
-      effort="20"
+      effort="200"
       velocity="6" />
   </joint>
@@ -218,5 +218,5 @@
       lower="0"
       upper="0.4754"
-      effort="20"
+      effort="200"
       velocity="6" />
   </joint>
@@ -274,7 +274,7 @@
       xyz="0 1 0" />
     <limit
-      lower="-0.185"
-      upper="0.185"
-      effort="20"
+      lower="-0.2"
+      upper="0.2"
+      effort="200"
       velocity="6" />
   </joint>
@@ -333,6 +333,6 @@
     <limit
       lower="0"
-      upper="3.14"
-      effort="20"
+       upper="3.14"
+      effort="200"
       velocity="6" />
   </joint>
@@ -390,7 +390,7 @@
       xyz="0 0 -1" />
     <limit
-      lower="-1.57"
+       lower="-1.57"
       upper="1.57"
-      effort="20"
+      effort="200"
       velocity="6" />
   </joint>
@@ -450,7 +450,13 @@
       lower="-1.57"
       upper="1.57"
-      effort="20"
-      velocity="6" />
-  </joint>
+      effort="100"
+      velocity="12" />
+  </joint>
+    <link name="world" />
+    <joint name="world_joint" type="fixed">
+      <parent link="world" />
+      <child link = "arm_base_link" />
+      <origin xyz="0.0 0.0 0.0" rpy="0.0 0.0 0.0" />
+    </joint>
    </xacro:macro>
 </robot>

File: sp_description/urdf/engineer_manipulator/manipulator_transmission.xacro (robot description, xacro)
@@ -6,8 +6,8 @@
             <actuator name="${joint_name}_motor">
                 <mechanicalReduction>${mechanical_reduction}</mechanicalReduction>
-				<hardwareInterface>hardware_interface/EffortJointInterface</hardwareInterface>
+				<hardwareInterface>hardware_interface/PositionJointInterface</hardwareInterface>
             </actuator>
 			<joint name="${joint_name}">
-				<hardwareInterface>hardware_interface/EffortJointInterface</hardwareInterface>
+				<hardwareInterface>hardware_interface/PositionJointInterface</hardwareInterface>
 			</joint>
         </transmission>
@@ -19,5 +19,8 @@
 	<xacro:manipulator_transmission joint_name="joint5" mechanical_reduction="1"/>
     <xacro:manipulator_transmission joint_name="joint6" mechanical_reduction="1"/>
-    <xacro:manipulator_transmission joint_name="joint7" mechanical_reduction="599.99"/>
+    <xacro:manipulator_transmission joint_name="joint7" mechanical_reduction="1"/>
+        <gazebo>
+        <plugin name="gazebo_ros_control" filename="libgazebo_ros_control.so"/>
+    </gazebo>
     <!-- <gazebo>
         <plugin name="gazebo_ros_vacuum_gripper" filename="libgazebo_ros_vacuum_gripper.so">
@@ -39,5 +42,4 @@
         <ki>2.0</ki>
         <material>Gazebo/Grey</material>
-    </gazebo>
-	 -->
+    </gazebo> -->
 </robot>
